Commit message: rescaled arena and added few objects

File: rsc/arena/urdf/arena.urdf (robot description, URDF)
Before this commit: robot arena, 8 links, 7 joints
Links:
- link boundary: geometry collision box size=0.0795 34.97837 1.58993; collision box size=0.0795 34.97837 1.58993
- link field_1: geometry collision box size=36.29588 34.78526 0.01431; visual mesh filename=../meshes/dae/Field.001.dae scale=3.49784 4.70071 4.76978
- link field_1_3: geometry collision box size=2.34629 0.24 2.4; collision box size=2.34629 0.24 2.4
- link field_1_4: geometry collision box size=2.25478 0.24 2.4; collision box size=2.25478 0.24 2.4
- link field_1_5: geometry collision box size=2.44621 0.24 2.4; collision box size=2.44621 0.24 2.4
- link field_1_6: geometry collision box size=2.54062 0.24 2.4; collision box size=2.54062 0.24 2.4
- link field_1_9: geometry visual mesh filename=../meshes/dae/Lines.002.dae scale=3.17985 4.76978 4.76978; visual mesh filename=../meshes/dae/Lines.dae scale=3.17985 4.76978 4.76978
Joints:
- joint boundary: origin xyz=0 0 -0.22 rpy=0 0 0 -> xyz=0 0 -0.264 rpy=0 0 0
- joint field_1_10_fixing: origin xyz=0 0.25919 0.12725 rpy=0 0 0 -> xyz=0 0.31103 0.1527 rpy=0 0 0
- joint field_1_3_fixing: origin xyz=10.30401 0 0.85994 rpy=0 0 0 -> xyz=12.36481 0 1.03193 rpy=0 0 0
- joint field_1_4_fixing: origin xyz=0 -10.15281 0.85994 rpy=0 0 -1.57 -> xyz=0 -12.18337 1.03193 rpy=0 0 -1.57
- joint field_1_5_fixing: origin xyz=-10.21168 0 0.85994 rpy=0 0 0 -> xyz=-12.25401 0 1.03193 rpy=0 0 0
- joint field_1_6_fixing: origin xyz=0 10.71017 0.85994 rpy=0 0 -1.57 -> xyz=0 12.8522 1.03193 rpy=0 0 -1.57
- joint field_1_9_fixing: origin xyz=0 0.25919 0.12725 rpy=0 0 0 -> xyz=0 0.31103 0.1527 rpy=0 0 0

Commit message: added objects

File: rsc/arena/urdf/arena.urdf (robot description, URDF)
Before this commit: robot arena, 8 links, 7 joints
Links:
- link field_1_3: geometry collision box size=2.34629 0.24 2.4; collision box size=2.34629 0.24 2.4
- link field_1_4: geometry collision box size=2.25478 0.24 2.4; collision box size=2.25478 0.24 2.4
- link field_1_5: geometry collision box size=2.44621 0.24 2.4; collision box size=2.44621 0.24 2.4
- link field_1_6: geometry collision box size=2.54062 0.24 2.4; collision box size=2.54062 0.24 2.4

Commit message: Updated

File: rsc/arena/urdf/arena.urdf (robot description, URDF)
Before this commit: robot arena, 8 links, 7 joints
Links:
- added link new_link, mass 0.001; visual mesh filename=../meshes/dae/Goalsallyback.001.dae scale=3.35214 1.58993 1.58993; visual mesh filename=../meshes/dae/Goalsallyback.dae scale=3.22758 1.58993 1.58993
- link field_1_3: geometry collision box size=2.34629 0.24 2.4; collision box size=2.34629 0.24 2.4
- link field_1_4: geometry collision box size=2.25478 0.24 2.4; collision box size=2.25478 0.24 2.4
- link field_1_5: geometry collision box size=2.44621 0.24 2.4; collision box size=2.44621 0.24 2.4
- link field_1_6: geometry collision box size=2.54062 0.24 2.4; collision box size=2.54062 0.24 2.4
Joints:
- added joint new_link: type floating, parent field_1, child new_link, origin xyz=0.31985 -0.37254 0.0176 rpy=0 0 0
